Commit message: added changes to devcontainer/dockerfile to ensure vcxsrv runs correctly; began slowly correcting rover arm urdf for rviz simulation

File: src/rover_arm/urdf/ASY, ROBOTIC ARM, 2026, URDF.urdf (robot description, URDF)
Before this commit: robot ASY, ROBOTIC ARM, 2026, URDF, 7 links, 6 joints
Links:
- added link world
- link End_effector: geometry collision mesh filename=package://rover_arm/meshes/End_effector.STL; visual mesh filename=package://rover_arm/meshes/End_effector.STL
- link Link1.5: geometry collision mesh filename=package://rover_arm/meshes/Link1.5.STL; visual mesh filename=package://rover_arm/meshes/Link1.5.STL
- link Link2: geometry collision mesh filename=package://rover_arm/meshes/Link2.STL; visual mesh filename=package://rover_arm/meshes/Link2.STL
- link Link3: geometry collision mesh filename=package://rover_arm/meshes/Link3.STL; visual mesh filename=package://rover_arm/meshes/Link3.STL
- link Link4: geometry collision mesh filename=package://rover_arm/meshes/Link4.STL; visual mesh filename=package://rover_arm/meshes/Link4.STL
- link Link5: geometry collision mesh filename=package://rover_arm/meshes/Link5.STL; visual mesh filename=package://rover_arm/meshes/Link5.STL
- link base_link: geometry collision mesh filename=package://rover_arm/meshes/base_link.STL; visual mesh filename=package://rover_arm/meshes/base_link.STL
Joints:
- added joint world_to_base: type fixed, parent world, child base_link, origin xyz=0 0 0 rpy=3.1416 0 0
