Commit message: added limits to robot arm range

File: src/rover_arm/urdf/rover_arm.urdf (robot description, URDF)
Before this commit: robot Rover_Arm, 8 links, 7 joints
Joints:
- joint wrist_roll_joint: limit lower=-1.5708 upper=1.5708 effort=10 velocity=1.0 -> lower=0 upper=3.1416 effort=10 velocity=1.0
